File: Titulador.sch (KiCad schematic (older format))
At the start: 28 parts, among them J1 1x2_F, J2 1x6_F, J3 1x4_F, J4 1x2_F, J5 1x5_F, J6 1x2_F, J7 1x4_F, Q1 BC548, SW1 SW_DIP_x03, U1 ESP32-DEVKITC-32D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

Commit message: Se agrega PCB
Parts:
- removed SW1: SW_DIP_x03, symbol Switch:SW_DIP_x03
- added SW1: SW_DIP_x04, Button_Switch_THT:SW_DIP_SPSTx04_Slide_6.7x11.72mm_W7.62mm_P2.54mm_LowProfile, symbol Switch:SW_DIP_x04
- C1: footprint (none) -> Capacitor_THT:CP_Radial_D7.5mm_P2.50mm
- D1: footprint (none) -> Diode_THT:D_A-405_P7.62mm_Horizontal
- J1, J4, J6: footprint (none) -> Connector_PinSocket_2.54mm:PinSocket_1x02_P2.54mm_Vertical
- J2: footprint (none) -> Connector_PinSocket_2.54mm:PinSocket_1x06_P2.54mm_Vertical
- J3, J7: footprint (none) -> Connector_PinSocket_2.54mm:PinSocket_1x04_P2.54mm_Vertical
- J5: footprint (none) -> Connector_PinSocket_2.54mm:PinSocket_1x05_P2.54mm_Vertical
- Q1: footprint Package_TO_SOT_THT:TO-92_Inline -> Package_TO_SOT_THT:TO-92L_HandSolder
- R1, R10, R11, R12, R13, R2, R3, R4, R5, R6, R7, R8, R9: footprint (none) -> Resistor_THT:R_Axial_DIN0207_L6.3mm_D2.5mm_P7.62mm_Horizontal
- U1: footprint MODULE_ESP32-DEVKITC-32D -> pcbTitulador:MODULE_ESP32-DEVKITC-32D; symbol ESP32-DEVKITC-32D:ESP32-DEVKITC-32D -> Titulador-rescue:ESP32-DEVKITC-32D-ESP32-DEVKITC-32D
- U2: footprint (none) -> pcbTitulador:MCUFriend; symbol MCU_Friend:MCU_Friend -> Titulador-rescue:MCU_Friend-MCU_Friend
Connections:
- net +3V3: now also U2.27 (3.3V); no longer U2.3.3V
- net +5V: now also U2.26 (5V), SW1.1, SW1.2, SW1.3; no longer U2.5V
- net GND: now also U2.24 (GND); no longer U2.GND
- net HCLK: now also U2.14 (SD_SCK); no longer U2.SCK (SD_SCK)
- net HCSO: now also U2.11 (SD_SS); no longer U2.SS (SD_SS)
- net HMISO: now also U2.13 (SD_MISO); no longer U2.SDO (SD_MISO)
- net HMOSI: now also U2.12 (SD_MOSI); no longer U2.SDI (SD_MOSI)
- net at A1.10 (M0): now also SW1.8
- net at A1.11 (M1): now also SW1.7
- net at A1.12 (M2): now also SW1.6
- net at A2.10 (D7): now also U2.8 (LCD_D7); no longer U2.D7 (LCD_D7)
- net at A2.11 (D8): now also U2.9 (LCD_D0); no longer U2.D0 (LCD_D0)
- net at A2.12 (D9): now also U2.10 (LCD_D1); no longer U2.D1 (LCD_D1)
- net at A2.19 (A0): now also U2.22 (LCD_RD); no longer U2.RD (LCD_RD)
- net at A2.20 (A1): now also U2.21 (LCD_WR); no longer U2.WR (LCD_WR)
- net at A2.21 (A2): now also U2.20 (LCD_RS); no longer U2.RS (LCD_RS)
- net at A2.22 (A3): now also U2.19 (LCD_CS); no longer U2.CS (LCD_CS)
- net at A2.23 (A4): now also U2.18 (LCD_RST); no longer U2.RST (LCD_RST)
- net at A2.5 (D2): now also U2.3 (LCD_D2); no longer U2.D2 (LCD_D2)
- net at A2.6 (D3): now also U2.4 (LCD_D3); no longer U2.D3 (LCD_D3)
- net at A2.7 (D4): now also U2.5 (LCD_D4); no longer U2.D4 (LCD_D4)
- net at A2.8 (D5): now also U2.6 (LCD_D5); no longer U2.D5 (LCD_D5)
- net at A2.9 (D6): now also U2.7 (LCD_D6); no longer U2.D6 (LCD_D6)
- no-connect marks 20 -> 22
Changed lines of the file:
@@
 $EndDescr
 $Comp
-L ESP32-DEVKITC-32D:ESP32-DEVKITC-32D U1
+L Titulador-rescue:ESP32-DEVKITC-32D-ESP32-DEVKITC-32D U1
 U 1 1 5F56BE4D
 P 4700 3850
 F 0 "U1" H 4700 5017 50  0000 C CNN
 F 1 "ESP32-DEVKITC-32D" H 4700 4926 50  0000 C CNN
-F 2 "MODULE_ESP32-DEVKITC-32D" H 4700 3850 50  0001 L BNN
+F 2 "pcbTitulador:MODULE_ESP32-DEVKITC-32D" H 4700 3850 50  0001 L BNN
 F 3 "4" H 4700 3850 50  0001 L BNN
 F 4 "Espressif Systems" H 4700 3850 50  0001 L BNN "Field4"
@@
 F 0 "R2" V 2265 2850 50  0000 C CNN
 F 1 "18K" V 2356 2850 50  0000 C CNN
-F 2 "" V 2080 2850 50  0001 C CNN
+F 2 "Resistor_THT:R_Axial_DIN0207_L6.3mm_D2.5mm_P7.62mm_Horizontal" V 2080 2850 50  0001 C CNN
 F 3 "~" H 2150 2850 50  0001 C CNN
 	1    2150 2850
@@
 F 0 "R5" H 2720 3096 50  0000 L CNN
 F 1 "27K" H 2720 3005 50  0000 L CNN
-F 2 "" V 2580 3050 50  0001 C CNN
+F 2 "Resistor_THT:R_Axial_DIN0207_L6.3mm_D2.5mm_P7.62mm_Horizontal" V 2580 3050 50  0001 C CNN
 F 3 "~" H 2650 3050 50  0001 C CNN
 	1    2650 3050
@@
 F 0 "R9" V 4793 6800 50  0000 C CNN
 F 1 "10K" V 4884 6800 50  0000 C CNN
-F 2 "" V 4930 6800 50  0001 C CNN
+F 2 "Resistor_THT:R_Axial_DIN0207_L6.3mm_D2.5mm_P7.62mm_Horizontal" V 4930 6800 50  0001 C CNN
 F 3 "~" H 5000 6800 50  0001 C CNN
 	1    5000 6800
@@
 F 0 "R10" H 2420 4496 50  0000 L CNN
 F 1 "27K" H 2420 4405 50  0000 L CNN
-F 2 "" V 2280 4450 50  0001 C CNN
+F 2 "Resistor_THT:R_Axial_DIN0207_L6.3mm_D2.5mm_P7.62mm_Horizontal" V 2280 4450 50  0001 C CNN
 F 3 "~" H 2350 4450 50  0001 C CNN
 	1    2350 4450
@@
 F 0 "R11" V 2815 4150 50  0000 C CNN
 F 1 "18K" V 2906 4150 50  0000 C CNN
-F 2 "" V 2630 4150 50  0001 C CNN
+F 2 "Resistor_THT:R_Axial_DIN0207_L6.3mm_D2.5mm_P7.62mm_Horizontal" V 2630 4150 50  0001 C CNN
 F 3 "~" H 2700 4150 50  0001 C CNN
 	1    2700 4150
@@
 F 0 "R7" H 3020 3096 50  0000 L CNN
 F 1 "27K" H 3020 3005 50  0000 L CNN
-F 2 "" V 2880 3050 50  0001 C CNN
+F 2 "Resistor_THT:R_Axial_DIN0207_L6.3mm_D2.5mm_P7.62mm_Horizontal" V 2880 3050 50  0001 C CNN
 F 3 "~" H 2950 3050 50  0001 C CNN
 	1    2950 3050
@@
 F 0 "D1" V 5550 6150 50  0000 C CNN
 F 1 "1N4007" V 5650 6050 50  0000 C CNN
-F 2 "" H 5600 6300 50  0001 C CNN
+F 2 "Diode_THT:D_A-405_P7.62mm_Horizontal" H 5600 6300 50  0001 C CNN
 F 3 "~" H 5600 6300 50  0001 C CNN
 	1    5600 6300
@@
 F 0 "Q1" H 5691 6846 50  0000 L CNN
 F 1 "BC548" H 5691 6755 50  0000 L CNN
-F 2 "Package_TO_SOT_THT:TO-92_Inline" H 5700 6725 50  0001 L CIN
+F 2 "Package_TO_SOT_THT:TO-92L_HandSolder" H 5700 6725 50  0001 L CIN
 F 3 "http://www.fairchildsemi.com/ds/BC/BC547.pdf" H 5500 6800 50  0001 L CNN
 	1    5500 6800
@@
 F 0 "J2" H 1292 2935 50  0000 C CNN
 F 1 "1x6_F" H 1292 2844 50  0000 C CNN
-F 2 "" H 1400 2550 50  0001 C CNN
+F 2 "Connector_PinSocket_2.54mm:PinSocket_1x06_P2.54mm_Vertical" H 1400 2550 50  0001 C CNN
 F 3 "~" H 1400 2550 50  0001 C CNN
 	1    1400 2550
@@
 F 0 "J3" H 3442 6225 50  0000 C CNN
 F 1 "1x4_F" H 3442 6316 50  0000 C CNN
-F 2 "" H 3550 6650 50  0001 C CNN
+F 2 "Connector_PinSocket_2.54mm:PinSocket_1x04_P2.54mm_Vertical" H 3550 6650 50  0001 C CNN
 F 3 "~" H 3550 6650 50  0001 C CNN
 	1    3550 6650
@@
 F 0 "C1" H 1618 5996 50  0000 L CNN
 F 1 "100uF" H 1618 5905 50  0000 L CNN
-F 2 "" H 1538 5800 50  0001 C CNN
+F 2 "Capacitor_THT:CP_Radial_D7.5mm_P2.50mm" H 1538 5800 50  0001 C CNN
 F 3 "~" H 1500 5950 50  0001 C CNN
 	1    1500 5950
 	-1   0    0    -1
-$EndComp
-$Comp
-L Switch:SW_DIP_x03 SW1
-U 1 1 5F57DE7B
-P 1350 7100
-F 0 "SW1" H 1350 6925 50  0000 C CNN
-F 1 "SW_DIP_x03" H 1350 6834 50  0000 C CNN
-F 2 "" H 1350 7100 50  0001 C CNN
-F 3 "~" H 1350 7100 50  0001 C CNN
-	1    1350 7100
-	1    0    0    -1
 $EndComp
 $Comp
@@
 F 0 "J4" H 1192 1235 50  0000 C CNN
 F 1 "1x2_F" H 1350 1150 50  0000 C CNN
-F 2 "" H 1300 1050 50  0001 C CNN
+F 2 "Connector_PinSocket_2.54mm:PinSocket_1x02_P2.54mm_Vertical" H 1300 1050 50  0001 C CNN
 F 3 "~" H 1300 1050 50  0001 C CNN
 	1    1300 1050
@@
 F 0 "J6" H 6300 6500 50  0000 L CNN
 F 1 "1x2_F" H 6100 6200 50  0000 L CNN
-F 2 "" H 6400 6350 50  0001 C CNN
+F 2 "Connector_PinSocket_2.54mm:PinSocket_1x02_P2.54mm_Vertical" H 6400 6350 50  0001 C CNN
 F 3 "~" H 6400 6350 50  0001 C CNN
 	1    6400 6350
@@
 F 0 "R1" V 1943 2650 50  0000 C CNN
 F 1 "18K" V 2034 2650 50  0000 C CNN
-F 2 "" V 2080 2650 50  0001 C CNN
+F 2 "Resistor_THT:R_Axial_DIN0207_L6.3mm_D2.5mm_P7.62mm_Horizontal" V 2080 2650 50  0001 C CNN
 F 3 "~" H 2150 2650 50  0001 C CNN
 	1    2150 2650
@@
 F 0 "J1" H 1242 1935 50  0000 C CNN
 F 1 "1x2_F" H 1242 1844 50  0000 C CNN
-F 2 "" H 1350 1750 50  0001 C CNN
+F 2 "Connector_PinSocket_2.54mm:PinSocket_1x02_P2.54mm_Vertical" H 1350 1750 50  0001 C CNN
 F 3 "~" H 1350 1750 50  0001 C CNN
 	1    1350 1750
@@
 F 0 "R6" V 2915 1850 50  0000 C CNN
 F 1 "18K" V 3006 1850 50  0000 C CNN
-F 2 "" V 2730 1850 50  0001 C CNN
+F 2 "Resistor_THT:R_Axial_DIN0207_L6.3mm_D2.5mm_P7.62mm_Horizontal" V 2730 1850 50  0001 C CNN
 F 3 "~" H 2800 1850 50  0001 C CNN
 	1    2800 1850
@@
 F 0 "R3" V 2043 1750 50  0000 C CNN
 F 1 "18K" V 2134 1750 50  0000 C CNN
-F 2 "" V 2180 1750 50  0001 C CNN
+F 2 "Resistor_THT:R_Axial_DIN0207_L6.3mm_D2.5mm_P7.62mm_Horizontal" V 2180 1750 50  0001 C CNN
 F 3 "~" H 2250 1750 50  0001 C CNN
 	1    2250 1750
@@
 F 0 "R8" H 3220 2146 50  0000 L CNN
 F 1 "27K" H 3220 2055 50  0000 L CNN
-F 2 "" V 3080 2100 50  0001 C CNN
+F 2 "Resistor_THT:R_Axial_DIN0207_L6.3mm_D2.5mm_P7.62mm_Horizontal" V 3080 2100 50  0001 C CNN
 F 3 "~" H 3150 2100 50  0001 C CNN
 	1    3150 2100
@@
 F 0 "R4" H 2570 2146 50  0000 L CNN
 F 1 "27K" H 2570 2055 50  0000 L CNN
-F 2 "" V 2430 2100 50  0001 C CNN
+F 2 "Resistor_THT:R_Axial_DIN0207_L6.3mm_D2.5mm_P7.62mm_Horizontal" V 2430 2100 50  0001 C CNN
 F 3 "~" H 2500 2100 50  0001 C CNN
 	1    2500 2100
@@
 	8500 3150 9800 3150
 $Comp
-L MCU_Friend:MCU_Friend U2
+L Titulador-rescue:MCU_Friend-MCU_Friend U2
 U 1 1 5F829702
 P 10200 3350
 F 0 "U2" H 10600 3200 50  0000 C CNN
 F 1 "MCU_Friend" H 10700 3400 50  0000 C CNN
-F 2 "" H 10300 3350 50  0001 C CNN
+F 2 "pcbTitulador:MCUFriend" H 10300 3350 50  0001 C CNN
 F 3 "" H 10300 3350 50  0001 C CNN
 	1    10200 3350
@@
 F 0 "J5" H 1292 4135 50  0000 C CNN
 F 1 "1x5_F" H 1292 4044 50  0000 C CNN
-F 2 "" H 1400 3750 50  0001 C CNN
+F 2 "Connector_PinSocket_2.54mm:PinSocket_1x05_P2.54mm_Vertical" H 1400 3750 50  0001 C CNN
 F 3 "~" H 1400 3750 50  0001 C CNN
 	1    1400 3750
@@
 F 0 "J7" H 5950 3950 50  0000 L CNN
 F 1 "1x4_F" H 5900 3850 50  0000 L CNN
-F 2 "" H 5900 4150 50  0001 C CNN
+F 2 "Connector_PinSocket_2.54mm:PinSocket_1x04_P2.54mm_Vertical" H 5900 4150 50  0001 C CNN
 F 3 "~" H 5900 4150 50  0001 C CNN
 	1    5900 4150
@@
 F 0 "R13" H 6370 3846 50  0000 L CNN
 F 1 "27K" H 6370 3755 50  0000 L CNN
-F 2 "" V 6230 3800 50  0001 C CNN
+F 2 "Resistor_THT:R_Axial_DIN0207_L6.3mm_D2.5mm_P7.62mm_Horizontal" V 6230 3800 50  0001 C CNN
 F 3 "~" H 6300 3800 50  0001 C CNN
 	1    6300 3800
@@
 F 0 "R12" V 5643 3650 50  0000 C CNN
 F 1 "18K" V 5734 3650 50  0000 C CNN
-F 2 "" V 5780 3650 50  0001 C CNN
+F 2 "Resistor_THT:R_Axial_DIN0207_L6.3mm_D2.5mm_P7.62mm_Horizontal" V 5780 3650 50  0001 C CNN
 F 3 "~" H 5850 3650 50  0001 C CNN
 	1    5850 3650
@@
 Wire Wire Line
 	5600 7000 5600 7200
+$Comp
+L Switch:SW_DIP_x04 SW1
+U 1 1 5F92A150
+P 1350 7100
+F 0 "SW1" H 1350 7567 50  0000 C CNN
+F 1 "SW_DIP_x04" H 1350 7476 50  0000 C CNN
+F 2 "Button_Switch_THT:SW_DIP_SPSTx04_Slide_6.7x11.72mm_W7.62mm_P2.54mm_LowProfile" H 1350 7100 50  0001 C CNN
+F 3 "~" H 1350 7100 50  0001 C CNN
+	1    1350 7100
+	1    0    0    -1
+$EndComp
+NoConn ~ 1050 7200
+NoConn ~ 1650 7200
 $EndSCHEMATC
